File: Lighting/Lighting.sch (KiCad schematic (older format))
At the start: 73 parts, among them J1 USB_C_Receptacle, J2 USB_C_Receptacle, Q1 PSMN011, U1 MCP2210T-I_SO, U2 UTC2000-I_MG, U3 DAC8551IDGKT, U4 LMC6482, U5 MCP1501_2v5, Y1 Crystal_12MHz

Commit message: finish PCB layout and output gerber
Parts:
- removed J_VDD1: TestPoint, wsolar:TP, symbol wsolar:TestPoint
- added unit 2 of U4
- added unit 3 of U4
- JP1: footprint (none) -> wsolar:jumper_2
- renumbered Vsink1 to Vs1
Connections:
- net labels added: VCC
- net labels removed: VDD
- wire segments 261 -> 275
- no-connect marks 37 -> 38
Other:
- note added: "Priotized Soldering"

Commit message: changes based on feedback
Parts:
- removed C8: C_0u1, wsolar:C_0805, symbol wsolar:C_0u1
- removed D1, D2, D3, D4: LED_645nm, wsolar:LED0805, symbol wsolar:LED_645nm
- removed J2: USB_C_Receptacle, wsolar:MOLEX_105450-0101, symbol wsolar:USB_C_Receptacle
- removed JP3, JP4: Jumper_NO_Small, wsolar:jumper_2, symbol wsolar:Jumper_NO_Small
- removed R10, R12, R8, R9: R_1k, wsolar:R0805, symbol wsolar:R_1k
- removed R14, R15, R6, R7: R_10k, wsolar:R0805, symbol wsolar:R_10k
- removed R17: R_39k4, wsolar:R0805, symbol wsolar:R_39k4
- removed R4: R_35k7, wsolar:R0805, symbol wsolar:R_35k7
- removed R5: R_5k1, wsolar:R0805, symbol wsolar:R_5k1
- removed U2: UTC2000-I_MG, wsolar:QFN50P300X300X90-17N, symbol wsolar:UTC2000-I_MG
- removed U3: DAC8551IDGKT, wsolar:S-PDSO-G8, symbol wsolar:DAC8551IDGKT
- added D1, D2: D_Zener_5v6, wsolar:SOD123, symbol wsolar:D_Zener_5v6
- added J2: USB_B_Micro, wsolar:FCI_10118193-0001LF, symbol wsolar:USB_B_Micro
- added JP3: Jumper_3, wsolar:jumper_3, symbol wsolar:Jumper_3
- added R4: R_10k, wsolar:R0805, symbol wsolar:R_10k
- added R5: R_39k2, wsolar:R0805, symbol wsolar:R_39k2
- added U3: DAC6551AQDGKRQ1, wsolar:SOP65P490X110-9N, symbol wsolar:DAC6551AQDGKRQ1
- C1, C10, C14, C15, C17, C18, C19, C2, C20, C6, C9: Unit Price (none) -> 0.20
- C11, R16: Unit Price (none) -> 0.21
- C12, C16: Unit Price (none) -> 0.13
- C13, C21, C7: Unit Price (none) -> 0.63
- C3, C4: Unit Price (none) -> 0.15
- D5, D6, D8: Unit Price (none) -> 0.26
- D7: Unit Price (none) -> 2.06
- J1, RV1: Unit Price (none) -> 2.15
- Q1: Unit Price (none) -> 0.50
- R1, R13, R20, R23: Unit Price (none) -> 0.36
- R11: Unit Price (none) -> 0.28
- R18, R19, R21, R22: Unit Price (none) -> 0.71
- R2, R3: Unit Price (none) -> 0.25
- U1: Unit Price (none) -> 1.94
- U4: Unit Price (none) -> 1.89
- U5: Unit Price (none) -> 0.78
- Y1: Unit Price (none) -> 0.72
Connections:
- wire segments 275 -> 215
- no-connect marks 38 -> 24

Commit message: fix 1u cap link mistake; give mcp2210 correct name
Parts:
- removed U1: MCP2210T-I_SO, wsolar:SOIC127P1030X265-20N, symbol wsolar:MCP2210T-I_SO
- added U1: MCP2210T-I_SS, wsolar:SOIC127P1030X265-20N, symbol wsolar:MCP2210T-I_SS
Changed lines of the file:
@@
 EESchema Schematic File Version 4
-LIBS:Lighting-cache
 EELAYER 26 0
 EELAYER END
@@
 $EndComp
 $Comp
-L wsolar:MCP2210T-I_SO U1
-U 1 1 5E8DDE22
-P 3800 7800
-F 0 "U1" H 3800 8765 50  0000 C CNN
-F 1 "MCP2210T-I_SO" H 3800 8674 50  0000 C CNN
-F 2 "wsolar:SOIC127P1030X265-20N" H 3800 7800 50  0001 L BNN
-F 3 "http://ww1.microchip.com/downloads/en/DeviceDoc/22288A.pdf" H 3800 7800 50  0001 L BNN
-F 4 "MCP2210T-I/SS" H 3509 8722 50  0001 C CNN "Mfr. #"
-F 5 "https://www.digikey.com/product-detail/en/microchip-technology/MCP2210T-I-SS/MCP2210T-I-SSCT-ND/8628832" H 3609 8822 50  0001 C CNN "Link"
-F 6 "1.94" H 0   0   50  0001 C CNN "Unit Price"
-	1    3800 7800
-	1    0    0    -1
-$EndComp
-$Comp
 L wsolar:R_1k R20
 U 1 1 5EBABE25
@@
 	1    0    0    -1
 $EndComp
+$Comp
+L wsolar:MCP2210T-I_SS U1
+U 1 1 5F43B9FA
+P 3800 7800
+F 0 "U1" H 3800 8765 50  0000 C CNN
+F 1 "MCP2210T-I_SS" H 3800 8674 50  0000 C CNN
+F 2 "wsolar:SOIC127P1030X265-20N" H 3800 7800 50  0001 L BNN
+F 3 "http://ww1.microchip.com/downloads/en/DeviceDoc/22288A.pdf" H 3800 7800 50  0001 L BNN
+F 4 "MCP2210T-I/SS" H 3509 8722 50  0001 C CNN "Mfr. #"
+F 5 "https://www.digikey.com/product-detail/en/microchip-technology/MCP2210T-I-SS/MCP2210T-I-SSCT-ND/8628832" H 3609 8822 50  0001 C CNN "Link"
+F 6 "1.94" H 3709 8922 79  0001 C CNN "Unit Price"
+	1    3800 7800
+	1    0    0    -1
+$EndComp

Commit message: fix 39k2 resistor error
Parts:
- C10, C15, C19, C2, C20, C6: Link https://www.digikey.com/product-detail/en/kemet/C0805C104K5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 -> https://www.digikey.com/product-detail/en/kemet/C0805C105K5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
- R5: Mfr. # CRG0805F12K -> ERA-6AEB3922V
Changed lines of the file:
@@
 EESchema Schematic File Version 4
+LIBS:Lighting-cache
 EELAYER 26 0
 EELAYER END
@@
 F 3 "https://content.kemet.com/datasheets/KEM_C1023_X7R_AUTO_SMD.pdf" H 13825 5350 50  0001 C CNN
 F 4 "C0805C105K4RACAUTO" H 14025 5550 50  0001 C CNN "Mfr. #"
-F 5 "https://www.digikey.com/product-detail/en/kemet/C0805C104K5RACAUTO/399-6928-1-ND/3314438" H 13925 5450 50  0001 C CNN "Link"
+F 5 "https://www.digikey.com/product-detail/en/kemet/C0805C105K5RACAUTO/399-6928-1-ND/3314438" H 13925 5450 50  0001 C CNN "Link"
 F 6 "0.20" H 0   0   50  0001 C CNN "Unit Price"
 	1    13800 5250
@@
 F 3 "https://content.kemet.com/datasheets/KEM_C1023_X7R_AUTO_SMD.pdf" H 4375 2900 50  0001 C CNN
 F 4 "C0805C105K4RACAUTO" H 4575 3100 50  0001 C CNN "Mfr. #"
-F 5 "https://www.digikey.com/product-detail/en/kemet/C0805C104K5RACAUTO/399-6928-1-ND/3314438" H 4475 3000 50  0001 C CNN "Link"
+F 5 "https://www.digikey.com/product-detail/en/kemet/C0805C105K5RACAUTO/399-6928-1-ND/3314438" H 4475 3000 50  0001 C CNN "Link"
 F 6 "0.20" H 300 0   50  0001 C CNN "Unit Price"
 	1    4350 2800
@@
 F 3 "https://content.kemet.com/datasheets/KEM_C1023_X7R_AUTO_SMD.pdf" H 9175 7800 50  0001 C CNN
 F 4 "C0805C105K4RACAUTO" H 9375 8000 50  0001 C CNN "Mfr. #"
-F 5 "https://www.digikey.com/product-detail/en/kemet/C0805C104K5RACAUTO/399-6928-1-ND/3314438" H 9275 7900 50  0001 C CNN "Link"
+F 5 "https://www.digikey.com/product-detail/en/kemet/C0805C105K5RACAUTO/399-6928-1-ND/3314438" H 9275 7900 50  0001 C CNN "Link"
 F 6 "0.20" H 0   0   50  0001 C CNN "Unit Price"
 	1    9150 7700
@@
 F 3 "https://content.kemet.com/datasheets/KEM_C1023_X7R_AUTO_SMD.pdf" H 2275 7400 50  0001 C CNN
 F 4 "C0805C105K4RACAUTO" H 2475 7600 50  0001 C CNN "Mfr. #"
-F 5 "https://www.digikey.com/product-detail/en/kemet/C0805C104K5RACAUTO/399-6928-1-ND/3314438" H 2375 7500 50  0001 C CNN "Link"
+F 5 "https://www.digikey.com/product-detail/en/kemet/C0805C105K5RACAUTO/399-6928-1-ND/3314438" H 2375 7500 50  0001 C CNN "Link"
 F 6 "0.20" H 0   0   50  0001 C CNN "Unit Price"
 	1    2250 7300
@@
 F 3 "https://content.kemet.com/datasheets/KEM_C1023_X7R_AUTO_SMD.pdf" H 13525 6750 50  0001 C CNN
 F 4 "C0805C105K4RACAUTO" H 13725 6950 50  0001 C CNN "Mfr. #"
-F 5 "https://www.digikey.com/product-detail/en/kemet/C0805C104K5RACAUTO/399-6928-1-ND/3314438" H 13625 6850 50  0001 C CNN "Link"
+F 5 "https://www.digikey.com/product-detail/en/kemet/C0805C105K5RACAUTO/399-6928-1-ND/3314438" H 13625 6850 50  0001 C CNN "Link"
 F 6 "0.20" H 0   0   50  0001 C CNN "Unit Price"
 	1    13500 6650
@@
 F 3 "https://content.kemet.com/datasheets/KEM_C1023_X7R_AUTO_SMD.pdf" H 10525 4250 50  0001 C CNN
 F 4 "C0805C105K4RACAUTO" H 10725 4450 50  0001 C CNN "Mfr. #"
-F 5 "https://www.digikey.com/product-detail/en/kemet/C0805C104K5RACAUTO/399-6928-1-ND/3314438" H 10625 4350 50  0001 C CNN "Link"
+F 5 "https://www.digikey.com/product-detail/en/kemet/C0805C105K5RACAUTO/399-6928-1-ND/3314438" H 10625 4350 50  0001 C CNN "Link"
 F 6 "0.20" H 0   0   50  0001 C CNN "Unit Price"
 	1    10500 4150
@@
 F 2 "wsolar:R0805" V 12180 6700 50  0001 C CNN
 F 3 "https://industrial.panasonic.com/cdbs/www-data/pdf/RDM0000/AOA0000C307.pdf" V 12330 6700 50  0001 C CNN
-F 4 "CRG0805F12K" V 12430 6800 50  0001 C CNN "Mfr. #"
+F 4 "ERA-6AEB3922V" V 12430 6800 50  0001 C CNN "Mfr. #"
 F 5 "https://www.digikey.com/product-detail/en/panasonic-electronic-components/ERA-6AEB3922V/P39-2KDADKR-ND/3075510" V 12530 6900 50  0001 C CNN "Link"
 F 6 "0.34" V 12630 7000 79  0001 C CNN "Unit Price"
